File: hardware/rev-a/product-d1/kicad/cadenza-d1.kicad_sch (KiCad schematic)
At the start: 59 parts, among them J1 USB-C USB2 Sink, J2 LS027B7DH01 FPC, J3 microSD push-push, J4 LiPo 1S, J5 Speaker 8R 1-2W, J6 Encoder daughterboard, SW1 POWER RUN/OFF, SW2 B, SW3 MENU, SW4 RESET, SW5 BOOT, U1 ESP32-S3-WROOM-1-N16R8, U2 BQ24074RGTR, U3 TPS63070RNMR, U4 TPS61023DRLR, U5 MAX98357AETE+T, U6 IM73D122V01, U7 BQ27441DRZR-G1A, U8 USBLC6-2SC6

Commit message: wip: add capability mode JSON, update circuit and component documentation for Rev A
Parts:
- added C11, C20, C50, C81, C90: 10uF, Capacitor_SMD:C_0603_1608Metric, symbol Cadenza_D1:PASSIVE
- added C12, C13, C21, C22: 22uF, Capacitor_SMD:C_0603_1608Metric, symbol Cadenza_D1:PASSIVE
- added C14, C31, C40, C51, C82, C91: 100nF, Capacitor_SMD:C_0603_1608Metric, symbol Cadenza_D1:PASSIVE
- added C30, C70, C71, C80: 1uF, Capacitor_SMD:C_0603_1608Metric, symbol Cadenza_D1:PASSIVE
- added FB1, FB2: 600R@100MHz, Inductor_SMD:L_0603_1608Metric, symbol Cadenza_D1:PASSIVE
- added L1, L2: 1uH Isat7.5A, Inductor_SMD:L_1210_3225Metric, symbol Cadenza_D1:PASSIVE
- C1: renamed from L1; value 1.2uH Isat>=4.5A -> 10uF; footprint Inductor_SMD:L_1210_3225Metric -> Capacitor_SMD:C_0603_1608Metric; LCSC (none) -> C19702; MPN (none) -> CL10A106KP8NNNC
- C10: renamed from FB2; value 600R@100MHz -> 10uF; footprint Inductor_SMD:L_0603_1608Metric -> Capacitor_SMD:C_0603_1608Metric; LCSC (none) -> C19702; MPN (none) -> CL10A106KP8NNNC
- C2: renamed from L2; value 1uH Isat>=4.5A -> 10uF; footprint Inductor_SMD:L_1210_3225Metric -> Capacitor_SMD:C_0603_1608Metric; LCSC (none) -> C19702; MPN (none) -> CL10A106KP8NNNC
- C3: renamed from FB1; value 600R@100MHz -> 10uF; footprint Inductor_SMD:L_0603_1608Metric -> Capacitor_SMD:C_0603_1608Metric; LCSC (none) -> C19702; MPN (none) -> CL10A106KP8NNNC
- J1: LCSC (none) -> C2997435; MPN (none) -> HC-TYPE-C-16P-01A-G
- J2: LCSC (none) -> C324723; MPN (none) -> FH34SRJ-10S-0.5SH(99)
- J3: LCSC (none) -> C114218; MPN (none) -> DM3AT-SF-PEJM5
- J4, J5: LCSC (none) -> TBD; MPN (none) -> B2B-PH-SM4-TB
- J6: LCSC (none) -> TBD; MPN (none) -> SM06B-SRSS-TB
- R1: renamed from R20; value 732k -> 5.1k; LCSC (none) -> C23186; MPN (none) -> 0603WAF5101T5E
- R10: renamed from R73; value 0.01R 1% -> 470k; LCSC (none) -> C23178; MPN (none) -> 0603WAF4703T5E
- R11: renamed from R80; value 10k -> 150k; LCSC (none) -> C22807; MPN (none) -> 0603WAF1503T5E
- R2: renamed from R21; value 100k -> 5.1k; LCSC (none) -> C23186; MPN (none) -> 0603WAF5101T5E
- R20: renamed from C1; value 10uF -> 732k; footprint Capacitor_SMD:C_0603_1608Metric -> Resistor_SMD:R_0603_1608Metric; LCSC (none) -> C5159703; MPN (none) -> FRC0603F7323TS
- R21: renamed from C2; value 10uF -> 100k; footprint Capacitor_SMD:C_0603_1608Metric -> Resistor_SMD:R_0603_1608Metric; LCSC (none) -> C25803; MPN (none) -> 0603WAF1003T5E
- R3: renamed from R40; value 100R -> 1.5k; LCSC (none) -> C22843; MPN (none) -> 0603WAF1501T5E
- R30: renamed from C31; value 100nF -> 100k; footprint Capacitor_SMD:C_0603_1608Metric -> Resistor_SMD:R_0603_1608Metric; LCSC (none) -> C25803; MPN (none) -> 0603WAF1003T5E
- R4: renamed from R41; value 100k -> 1.2k; LCSC (none) -> C22765; MPN (none) -> 0603WAF1201T5E
- R40: renamed from C3; value 10uF -> 100R; footprint Capacitor_SMD:C_0603_1608Metric -> Resistor_SMD:R_0603_1608Metric; LCSC (none) -> C22775; MPN (none) -> 0603WAF1000T5E
- R41: renamed from C10; value 10uF -> 100k; footprint Capacitor_SMD:C_0603_1608Metric -> Resistor_SMD:R_0603_1608Metric; LCSC (none) -> C25803; MPN (none) -> 0603WAF1003T5E
- R5: renamed from R70; value 4.7k -> 1.5k; LCSC (none) -> C22843; MPN (none) -> 0603WAF1501T5E
- R6: renamed from R71; value 4.7k -> 47k; LCSC (none) -> C25819; MPN (none) -> 0603WAF4702T5E
- R7: renamed from R72; LCSC (none) -> C25804; MPN (none) -> 0603WAF1002T5E
- R70: renamed from C11; value 10uF -> 4.7k; footprint Capacitor_SMD:C_0603_1608Metric -> Resistor_SMD:R_0603_1608Metric; LCSC (none) -> C23162; MPN (none) -> 0603WAF4701T5E
- R71: renamed from C12; value 22uF -> 4.7k; footprint Capacitor_SMD:C_0603_1608Metric -> Resistor_SMD:R_0603_1608Metric; LCSC (none) -> C23162; MPN (none) -> 0603WAF4701T5E
- R72: renamed from C13; value 22uF -> 10k; footprint Capacitor_SMD:C_0603_1608Metric -> Resistor_SMD:R_0603_1608Metric; LCSC (none) -> C25804; MPN (none) -> 0603WAF1002T5E
- R73: renamed from C14; value 100nF -> 0.01R 1% 1W 50ppm; footprint Capacitor_SMD:C_0603_1608Metric -> Resistor_SMD:R_2512_6332Metric; LCSC (none) -> TBD; MPN (none) -> VALUE_TO_FREEZE
- R74: renamed from C20; value 10uF -> 10k; footprint Capacitor_SMD:C_0603_1608Metric -> Resistor_SMD:R_0603_1608Metric; LCSC (none) -> C25804; MPN (none) -> 0603WAF1002T5E
- R75: renamed from C21; value 22uF -> 100k; footprint Capacitor_SMD:C_0603_1608Metric -> Resistor_SMD:R_0603_1608Metric; LCSC (none) -> C25803; MPN (none) -> 0603WAF1003T5E
- R76: renamed from C22; value 22uF -> 100k; footprint Capacitor_SMD:C_0603_1608Metric -> Resistor_SMD:R_0603_1608Metric; LCSC (none) -> C25803; MPN (none) -> 0603WAF1003T5E
- R77: renamed from C30; value 1uF -> 100k; footprint Capacitor_SMD:C_0603_1608Metric -> Resistor_SMD:R_0603_1608Metric; LCSC (none) -> C25803; MPN (none) -> 0603WAF1003T5E
- R80: renamed from C80; value 1uF -> 10k; footprint Capacitor_SMD:C_0603_1608Metric -> Resistor_SMD:R_0603_1608Metric; LCSC (none) -> C25804; MPN (none) -> 0603WAF1002T5E
- R90: renamed from C40; value 100nF -> 10k; footprint Capacitor_SMD:C_0603_1608Metric -> Resistor_SMD:R_0603_1608Metric; LCSC (none) -> C25804; MPN (none) -> 0603WAF1002T5E
- R91: renamed from C50; value 10uF -> 10k; footprint Capacitor_SMD:C_0603_1608Metric -> Resistor_SMD:R_0603_1608Metric; LCSC (none) -> C25804; MPN (none) -> 0603WAF1002T5E
- R92: renamed from C51; value 100nF -> 10k; footprint Capacitor_SMD:C_0603_1608Metric -> Resistor_SMD:R_0603_1608Metric; LCSC (none) -> C25804; MPN (none) -> 0603WAF1002T5E
- R93: renamed from C70; value 1uF -> 10k; footprint Capacitor_SMD:C_0603_1608Metric -> Resistor_SMD:R_0603_1608Metric; LCSC (none) -> C25804; MPN (none) -> 0603WAF1002T5E
- SW1: LCSC (none) -> TBD; MPN (none) -> JS102011SAQN
- SW2, SW3, SW4, SW5: LCSC (none) -> TBD; MPN (none) -> KMR2
- TP1: renamed from R1; value 5.1k -> UART_TX; footprint Resistor_SMD:R_0603_1608Metric -> TestPoint:TestPoint_Pad_D1.0mm; symbol Cadenza_D1:PASSIVE -> Cadenza_D1:TESTPOINT; LCSC (none) -> N/A; MPN (none) -> PCB_TEST_PAD
- TP2: renamed from R2; value 5.1k -> UART_RX; footprint Resistor_SMD:R_0603_1608Metric -> TestPoint:TestPoint_Pad_D1.0mm; symbol Cadenza_D1:PASSIVE -> Cadenza_D1:TESTPOINT; LCSC (none) -> N/A; MPN (none) -> PCB_TEST_PAD
- TP3: renamed from R3; value 1.5k -> GND; footprint Resistor_SMD:R_0603_1608Metric -> TestPoint:TestPoint_Pad_D1.0mm; symbol Cadenza_D1:PASSIVE -> Cadenza_D1:TESTPOINT; LCSC (none) -> N/A; MPN (none) -> PCB_TEST_PAD
- TP4: renamed from R4; value 1.18k -> PG_3V3; footprint Resistor_SMD:R_0603_1608Metric -> TestPoint:TestPoint_Pad_D1.0mm; symbol Cadenza_D1:PASSIVE -> Cadenza_D1:TESTPOINT; LCSC (none) -> N/A; MPN (none) -> PCB_TEST_PAD
- TP5: renamed from R5; value 1.5k -> PACKP; footprint Resistor_SMD:R_0603_1608Metric -> TestPoint:TestPoint_Pad_D1.0mm; symbol Cadenza_D1:PASSIVE -> Cadenza_D1:TESTPOINT; LCSC (none) -> N/A; MPN (none) -> PCB_TEST_PAD
- TP6: renamed from R6; value 47k -> VBAT; footprint Resistor_SMD:R_0603_1608Metric -> TestPoint:TestPoint_Pad_D1.0mm; symbol Cadenza_D1:PASSIVE -> Cadenza_D1:TESTPOINT; LCSC (none) -> N/A; MPN (none) -> PCB_TEST_PAD
- TP7: renamed from R7; value 10k -> VSYS; footprint Resistor_SMD:R_0603_1608Metric -> TestPoint:TestPoint_Pad_D1.0mm; symbol Cadenza_D1:PASSIVE -> Cadenza_D1:TESTPOINT; LCSC (none) -> N/A; MPN (none) -> PCB_TEST_PAD
- TP8: renamed from R10; value 470k -> +3V3; footprint Resistor_SMD:R_0603_1608Metric -> TestPoint:TestPoint_Pad_D1.0mm; symbol Cadenza_D1:PASSIVE -> Cadenza_D1:TESTPOINT; LCSC (none) -> N/A; MPN (none) -> PCB_TEST_PAD
- TP9: renamed from R11; value 150k -> +5V; footprint Resistor_SMD:R_0603_1608Metric -> TestPoint:TestPoint_Pad_D1.0mm; symbol Cadenza_D1:PASSIVE -> Cadenza_D1:TESTPOINT; LCSC (none) -> N/A; MPN (none) -> PCB_TEST_PAD
- U1: LCSC (none) -> C2913202; MPN (none) -> ESP32-S3-WROOM-1-N16R8
- U2: LCSC (none) -> C54313; MPN (none) -> BQ24074RGTR
- U3: footprint Cadenza_D1:TI_RNM0015A_VQFN-HR-15_2.5x3mm -> Cadenza_D1:TI_RNM0015A_VQFN-HR-15_TI4222000B; LCSC (none) -> C109322; MPN (none) -> TPS63070RNMR
- U4: LCSC (none) -> C919459; MPN (none) -> TPS61023DRLR
- U5: LCSC (none) -> C910544; MPN (none) -> MAX98357AETE+T
- U6: LCSC (none) -> C5563886; MPN (none) -> IM73D122V01
- U7: footprint Cadenza_D1:TI_DRZ0012A_VSON-12_2.5x4mm -> Package_SON:Texas_S-PDSO-N12; LCSC (none) -> C473397; MPN (none) -> BQ27441DRZR-G1A
- U8: LCSC (none) -> C7519; MPN (none) -> USBLC6-2SC6
Connections:
- net +3V3_MAIN: now also R10.1, R41.2, R70.2, R71.2, R74.2, R75.2, R76.2, R77.2, R80.1, R90.2, R91.2, R92.2, R93.2, C12.1, C13.1, C40.1, C81.1, C82.1, C90.1, C91.1; no longer R11.1, R4.2, R5.2, R6.2, R71.1, R72.1, R90.1, U2.6 (EN1)
- net +5V_AUDIO: now also C50.1, C51.1, FB2.2; no longer C10.2, R91.1, R92.1
- net +5V_LCD: now also C30.1, C31.1, FB1.2; no longer C3.2, R30.1, R77.1
- net +5V_MEDIA: now also R20.1, TP9.1 (TP), C21.1, C22.1, FB1.1, FB2.1; no longer C10.1, C3.1, R1.1, R75.1, R76.1
- net AMP_EN: now also R41.1; no longer R4.1
- net BAT_TS: now also R7.1; no longer TP7.1
- net BOOST_SW: now also L2.2; no longer C2.2
- net CC1: now also R1.1; no longer TP1.1
- net CC2: now also R2.1; no longer TP2.1
- net CHG_N: now also R77.1
- net ESP_EN: now also R80.2, C80.1; no longer R11.2, R80.1
- net FB_3V3: now also R10.2, R11.1; no longer TP8.2, TP9.1
- net FB_5V: now also R20.2, R21.1; no longer R1.2, R2.1
- net GAUGE_BIN: now also R72.1, U7.10 (BIN); no longer R7.1, U7.9 (BIN)
- net GAUGE_INT_N: now also R74.1, U1.23 (GPIO21)
- net GAUGE_VDD: now also U7.5 (VDD), C71.1; no longer U7.2 (VDD)
- net GND: now also C1.2, C10.2, C2.2, C3.2, R1.2, R11.2, R3.2, R4.2, R5.2, R6.2, TP3.1 (TP), U7.3 (VSS), C11.2, C12.2, C13.2, C14.2, C20.2, C21.2, C22.2, C30.2, C31.2, C40.2, C50.2, C51.2, C70.2, C71.2, C80.2, C81.2, C82.2, C90.2, C91.2; no longer R20.2, R30.2, R40.2, R41.2, R70.2, R71.2, R73.2, R74.2, R75.2, R76.2, R77.2, R80.2, R90.2, R91.2, R92.2, R93.2, TP1.2, TP2.2, TP3.2, TP4.2, TP5.2, TP6.2, TP7.2, TP9.2, U7.4 (VSS)
- net I2C_SCL: now also R71.1, U7.2 (SCL); no longer R6.1, U7.5 (SCL)
- net I2C_SDA: now also R70.1; no longer R5.1
- net I2S_BCLK: now also U1.9 (GPIO16); no longer U1.16 (GPIO46)
- net ILIM_SET: now also R3.1; no longer TP3.1
- net ISET_SET: now also R4.1; no longer TP4.1
- net ITERM_SET: now also R5.1; no longer TP5.1
- net L3V3_A: now also L1.1; no longer C1.1
- net L3V3_B: now also L1.2; no longer C1.2
- net LED_CTRL: now also U1.38 (GPIO2)
- net PDM_DATA: now also R40.2; no longer R3.2
- net PDM_DATA_RAW: now also R40.1; no longer R3.1
- net PGOOD_N: now also R75.1, U1.39 (GPIO1)
- net PG_3V3_N: now also R76.1, TP4.1 (TP)
- net RUN_EN: now also R30.2
- net SD_CD: now also J3.9 (CD), R93.1, U1.17 (GPIO9); no longer U1.26 (GPIO45)
- net SD_CMD: now also R91.1
- net SD_CS: now also R90.1
- net SD_DAT0: now also R92.1
- net TMR_SET: now also R6.1; no longer TP6.1
- net UART_RX0: now also TP2.1 (TP)
- net UART_TX0: now also TP1.1 (TP)
- net VAUX_3V3: now also C14.1; no longer R73.1
- net VBAT: now also C3.1, R73.2, TP6.1 (TP), U7.7 (SRN); no longer J4.1 (P1), R40.1
- net VBUS: now also C1.1; no longer R20.1
- net VSYS: now also C10.1, R30.1, TP7.1 (TP), U2.6 (EN1), C11.1, C20.1, L2.1; no longer R21.1, R41.1, R70.1, R74.1
- net PACKP: now reaches U7.8 (SRP)
- net PACKP: now also J4.1 (P1), R73.1, TP5.1 (TP), U7.6 (BAT), C70.1
- removed net GAUGE_SRN: R10.2, U7.7 (SRN)
- net GAUGE_SRP: no longer names the net of U7.11 (NC)
- net GAUGE_SRP: no longer R10.1
- removed net VBAT_SENSE: R93.1, U7.6 (BAT)
- no-connect marks 18 -> 14
Other:
- moved on the sheet: C1, C10, C2, C3, R1, R10, R11, R2, R20, R21, R3, R30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
